Commit message: Remove unused xacro macro

File: src/cart_pole/cart_pole_bringup/urdf/macros.urdf.xacro (robot description, xacro)
@@ -8,10 +8,3 @@
     </inertial>
   </xacro:macro>
-  <xacro:macro name="cylinder_inertia" params="m r h xyz:='0.0 0.0 0.0' rpy:='0.0 0.0 0.0'">
-    <inertial>
-      <origin xyz="${xyz}" rpy="${rpy}"/>
-      <mass value="${m}"/>
-      <inertia ixx="${(m/12) * (3*r*r + h*h)}" ixy = "0" ixz = "0" iyy="${(m/12) * (3*r*r + h*h)}" iyz = "0" izz="${(m/2) * (r*r)}"/>
-    </inertial>
-  </xacro:macro>
 </robot>
