Commit message: Add genesis basic policy

File: src/cart_pole/cart_pole_bringup/urdf/cart_pole.urdf (robot description, URDF)
Before this commit: robot cart_pole, 4 links, 3 joints
Joints:
- removed joint slide_to_pole_with_holder
- added joint slider_to_pole_with_holder: type revolute, parent cart, child pole_with_holder, origin xyz=0.08 0 0 rpy=1.5707963267948966 0 0, axis 1 0 0, limit lower=-1.4 upper=1.4 effort=10000 velocity=1000
