Commit message: Add cart pole

File: src/cart_pole/cart_pole_bringup/urdf/cart_pole.urdf.xacro (robot description, xacro)
@@ -1,4 +1,11 @@
 <?xml version="1.0" ?>
-<robot name="cartopole">
+<robot name="cartopole" xmlns:xacro="http://ros.org/wiki/xacro">
+  <xacro:macro name="cylinder_inertia" params="m r h">
+    <inertial>
+      <origin xyz="0 0 0" rpy="${pi/2} 0 0" />
+      <mass value="${m}"/>
+      <inertia ixx="${(m/12) * (3*r*r + h*h)}" ixy = "0" ixz = "0" iyy="${(m/12) * (3*r*r + h*h)}" iyz = "0" izz="${(m/2) * (r*r)}"/>
+    </inertial>
+  </xacro:macro>
   <link name="world"/>
   <link name="slideBar">
@@ -19,11 +26,79 @@
         <box size="0.5 0.5 0.2"/>
       </geometry>
-      <origin xyz="0 0 1"/>
-    </visual>
-    <inertial>
-      <mass value="1"/>
-      <inertia ixx="1.0" ixy="0.0" ixz="0.0" iyy="1.0" iyz="0.0" izz="1.0"/>
-    </inertial>
-  </link>
+      <origin xyz="0 0 0"/>
+    </visual>
+    <inertial>
+      <mass value="1"/>
+      <inertia ixx="1.0" ixy="0.0" ixz="0.0" iyy="1.0" iyz="0.0" izz="1.0"/>
+    </inertial>
+  </link>
+  <link name="pole_holder">
+    <visual>
+      <origin xyz="0 0 0"/>
+      <geometry>
+        <box size="0.1 0.1 0.2"/>
+      </geometry>
+    </visual>
+    <collision>
+      <geometry>
+        <box size="0.1 0.1 0.2"/>
+      </geometry>
+      <origin xyz="0 0 0"/>
+    </collision>
+    <inertial>
+      <mass value="1"/>
+      <inertia ixx="1.0" ixy="0.0" ixz="0.0" iyy="1.0" iyz="0.0" izz="1.0"/>
+    </inertial>
+  </link>
+  <joint name="cart_to_pole_holder" type="fixed">
+    <origin xyz="0.0 0.0 0.2"/>
+    <parent link="cart"/>
+    <child link="pole_holder"/>
+  </joint>
+  <link name="pole_holder2">
+    <visual>
+      <geometry>
+        <cylinder radius="0.05" length="0.05"/>
+      </geometry>
+      <origin xyz="0 0.0 0.0" rpy="1.57 0.0 0.0"/>
+    </visual>
+    <collision>
+      <geometry>
+        <cylinder radius="0.05" length="0.05"/>
+      </geometry>
+      <origin xyz="0 0.0 0.0" rpy="1.57 0.0 0.0"/>
+    </collision>
+    <inertial>
+      <mass value="1.5"/>
+      <inertia ixx="1.0" ixy="0.0" ixz="0.0" iyy="1.0" iyz="0.0" izz="1.0"/>
+    </inertial>
+  </link>
+  <joint name="pole_holder_to_pole_holder2" type="revolute">
+    <axis xyz="0 1 0"/>
+    <origin xyz="0.0 0.075 0.05" rpy="0 0 0" />
+    <parent link="pole_holder"/>
+    <child link="pole_holder2"/>
+    <limit effort="10.0" lower="-5.0" upper="5.0" velocity="15.0"/>
+  </joint>
+  <link name="pole">
+    <visual>
+      <geometry>
+        <cylinder radius="0.05" length="0.5"/>
+      </geometry>
+      <origin xyz="0 0 0"/>
+    </visual>
+    <collision>
+      <geometry>
+        <cylinder radius="0.05" length="0.5"/>
+      </geometry>
+      <origin xyz="0 0 0"/>
+    </collision>
+    <xacro:cylinder_inertia m="5" r="0.05" h="0.5" />
+  </link>
+  <joint name="pole_holder_to_pole" type="fixed">
+    <origin xyz="0.0 0.075 0.15"/>
+    <parent link="pole_holder2"/>
+    <child link="pole"/>
+  </joint>
   <link name="leg1">
     <visual>
@@ -69,5 +144,5 @@
   <joint name="slider_to_cart" type="prismatic">
     <axis xyz="1 0 0"/>
-    <origin xyz="0.0 0.0 0.0"/>
+    <origin xyz="0.0 0.0 1.0"/>
     <parent link="slideBar"/>
     <child link="cart"/>
@@ -116,4 +191,8 @@
       <state_interface name="position"/>
     </joint>
+    <joint name="pole_holder_to_pole">
+      <state_interface name="velocity"/>
+      <state_interface name="position"/>
+    </joint>
   </ros2_control>
   <gazebo>

Commit message: Update limits for pole joint

File: src/cart_pole/cart_pole_bringup/urdf/cart_pole.urdf.xacro (robot description, xacro)
@@ -79,5 +79,5 @@
     <parent link="pole_holder"/>
     <child link="pole_holder2"/>
-    <limit effort="10.0" lower="-5.0" upper="5.0" velocity="15.0"/>
+    <limit effort="10.0" lower="-1.57" upper="1.57" velocity="15.0"/>
   </joint>
   <link name="pole">

Commit message: Enable collisions with limtiers

File: src/cart_pole/cart_pole_bringup/urdf/cart_pole.urdf.xacro (robot description, xacro)
@@ -12,5 +12,5 @@
     <visual>
       <geometry>
-        <box size="30 0.05 0.05"/>
+        <box size="10 0.05 0.05"/>
       </geometry>
       <origin xyz="0 0 1"/>
@@ -28,4 +28,10 @@
       <origin xyz="0 0 0"/>
     </visual>
+    <collision>
+      <geometry>
+        <box size="0.5 0.5 0.2"/>
+      </geometry>
+      <origin xyz="0 0 0"/>
+    </collision>
     <inertial>
       <mass value="1"/>
@@ -104,16 +110,16 @@
     <visual>
       <geometry>
-        <cylinder radius="0.2" length="1.0"/>
-      </geometry>
-      <origin xyz="0 0 0"/>
-    </visual>
-    <collision>
-      <geometry>
-        <cylinder radius="0.2" length="1.0"/>
-      </geometry>
-      <origin xyz="0 0 0"/>
-    </collision>
-    <inertial>
-      <mass value="1"/>
+        <cylinder radius="0.2" length="2.0"/>
+      </geometry>
+      <origin xyz="0 0 0"/>
+    </visual>
+    <collision>
+      <geometry>
+        <cylinder radius="0.2" length="2.0"/>
+      </geometry>
+      <origin xyz="0 0 0"/>
+    </collision>
+    <inertial>
+      <mass value="2"/>
       <inertia ixx="1.0" ixy="0.0" ixz="0.0" iyy="1.0" iyz="0.0" izz="1.0"/>
     </inertial>
@@ -122,16 +128,16 @@
     <visual>
       <geometry>
-        <cylinder radius="0.2" length="1.0"/>
-      </geometry>
-      <origin xyz="0 0 0"/>
-    </visual>
-    <collision>
-      <geometry>
-        <cylinder radius="0.2" length="1.0"/>
-      </geometry>
-      <origin xyz="0 0 0"/>
-    </collision>
-    <inertial>
-      <mass value="1"/>
+        <cylinder radius="0.2" length="2.0"/>
+      </geometry>
+      <origin xyz="0 0 0"/>
+    </visual>
+    <collision>
+      <geometry>
+        <cylinder radius="0.2" length="2.0"/>
+      </geometry>
+      <origin xyz="0 0 0"/>
+    </collision>
+    <inertial>
+      <mass value="2"/>
       <inertia ixx="1.0" ixy="0.0" ixz="0.0" iyy="1.0" iyz="0.0" izz="1.0"/>
     </inertial>
@@ -147,14 +153,14 @@
     <parent link="slideBar"/>
     <child link="cart"/>
-    <limit effort="1000.0" lower="-15" upper="15" velocity="30"/>
-    <dynamics damping="0.0" friction="0.0"/>
+    <limit effort="10.0" lower="-5" upper="5" velocity="30"/>
+    <dynamics damping="0.1" friction="0.1"/>
   </joint>
   <joint name="slider_to_leg1" type="fixed">
-    <origin xyz="-15.0 0.0 0.5"/>
+    <origin xyz="-5 0.0 1"/>
     <parent link="slideBar"/>
     <child link="leg1"/>
   </joint>
   <joint name="slider_to_leg2" type="fixed">
-    <origin xyz="15 0.0 0.5"/>
+    <origin xyz="5 0.0 1"/>
     <parent link="slideBar"/>
     <child link="leg2"/>
@@ -200,4 +206,5 @@
       <parameters>$(find cart_pole_bringup)/config/cart_pole_controllers.yaml</parameters>
     </plugin>
+    <self_collide>true</self_collide>
   </gazebo>
 </robot>

Commit message: Urdf refactor. Use floating point onnly when needed

File: src/cart_pole/cart_pole_bringup/urdf/cart_pole.urdf.xacro (robot description, xacro)
@@ -18,5 +18,5 @@
     <inertial>
       <mass value="100"/>
-      <inertia ixx="1.0" ixy="0.0" ixz="0.0" iyy="1.0" iyz="0.0" izz="1.0"/>
+      <inertia ixx="1" ixy="0" ixz="0" iyy="1" iyz="0" izz="1"/>
     </inertial>
   </link>
@@ -36,5 +36,5 @@
     <inertial>
       <mass value="1"/>
-      <inertia ixx="1.0" ixy="0.0" ixz="0.0" iyy="1.0" iyz="0.0" izz="1.0"/>
+      <inertia ixx="1" ixy="0" ixz="0" iyy="1" iyz="0" izz="1"/>
     </inertial>
   </link>
@@ -54,9 +54,9 @@
     <inertial>
       <mass value="1"/>
-      <inertia ixx="1.0" ixy="0.0" ixz="0.0" iyy="1.0" iyz="0.0" izz="1.0"/>
+      <inertia ixx="1" ixy="0" ixz="0" iyy="1" iyz="0" izz="1"/>
     </inertial>
   </link>
   <joint name="cart_to_pole_holder" type="fixed">
-    <origin xyz="0.0 0.0 0.2"/>
+    <origin xyz="0 0 0.2"/>
     <parent link="cart"/>
     <child link="pole_holder"/>
@@ -67,5 +67,5 @@
         <cylinder radius="0.05" length="0.05"/>
       </geometry>
-      <origin xyz="0 0.0 0.0" rpy="1.57 0.0 0.0"/>
+      <origin xyz="0 0 0" rpy="1.57 0 0"/>
     </visual>
     <collision>
@@ -73,17 +73,17 @@
         <cylinder radius="0.05" length="0.05"/>
       </geometry>
-      <origin xyz="0 0.0 0.0" rpy="1.57 0.0 0.0"/>
+      <origin xyz="0 0 0" rpy="1.57 0 0"/>
     </collision>
     <inertial>
       <mass value="1.5"/>
-      <inertia ixx="1.0" ixy="0.0" ixz="0.0" iyy="1.0" iyz="0.0" izz="1.0"/>
+      <inertia ixx="1" ixy="0" ixz="0" iyy="1" iyz="0" izz="1"/>
     </inertial>
   </link>
   <joint name="pole_holder_to_pole_holder2" type="revolute">
     <axis xyz="0 1 0"/>
-    <origin xyz="0.0 0.075 0.05" rpy="0 0 0" />
+    <origin xyz="0 0.075 0.05" rpy="0 0 0" />
     <parent link="pole_holder"/>
     <child link="pole_holder2"/>
-    <limit effort="10.0" lower="-1.57" upper="1.57" velocity="15.0"/>
+    <limit effort="10" lower="-1.57" upper="1.57" velocity="15"/>
   </joint>
   <link name="pole">
@@ -103,5 +103,5 @@
   </link>
   <joint name="pole_holder_to_pole" type="fixed">
-    <origin xyz="0.0 0.075 0.15"/>
+    <origin xyz="0 0.075 0.15"/>
     <parent link="pole_holder2"/>
     <child link="pole"/>
@@ -122,5 +122,5 @@
     <inertial>
       <mass value="2"/>
-      <inertia ixx="1.0" ixy="0.0" ixz="0.0" iyy="1.0" iyz="0.0" izz="1.0"/>
+      <inertia ixx="1" ixy="0" ixz="0" iyy="1" iyz="0" izz="1"/>
     </inertial>
   </link>
@@ -140,5 +140,5 @@
     <inertial>
       <mass value="2"/>
-      <inertia ixx="1.0" ixy="0.0" ixz="0.0" iyy="1.0" iyz="0.0" izz="1.0"/>
+      <inertia ixx="1" ixy="0" ixz="0" iyy="1" iyz="0" izz="1"/>
     </inertial>
   </link>
@@ -150,5 +150,5 @@
   <joint name="slider_to_cart" type="prismatic">
     <axis xyz="1 0 0"/>
-    <origin xyz="0.0 0.0 1.0"/>
+    <origin xyz="0 0 1.0"/>
     <parent link="slideBar"/>
     <child link="cart"/>
@@ -157,10 +157,10 @@
   </joint>
   <joint name="slider_to_leg1" type="fixed">
-    <origin xyz="-5 0.0 1"/>
+    <origin xyz="-5 0 1"/>
     <parent link="slideBar"/>
     <child link="leg1"/>
   </joint>
   <joint name="slider_to_leg2" type="fixed">
-    <origin xyz="5 0.0 1"/>
+    <origin xyz="5 0 1"/>
     <parent link="slideBar"/>
     <child link="leg2"/>

Commit message: Update pole params

File: src/cart_pole/cart_pole_bringup/urdf/cart_pole.urdf.xacro (robot description, xacro)
@@ -82,5 +82,5 @@
   <joint name="pole_holder_to_pole_holder2" type="revolute">
     <axis xyz="0 1 0"/>
-    <origin xyz="0 0.075 0.05" rpy="0 0 0" />
+    <origin xyz="0 0.075 0.05" rpy="0 0.001 0" />
     <parent link="pole_holder"/>
     <child link="pole_holder2"/>
@@ -90,15 +90,15 @@
     <visual>
       <geometry>
-        <cylinder radius="0.05" length="0.5"/>
-      </geometry>
-      <origin xyz="0 0 0"/>
-    </visual>
-    <collision>
-      <geometry>
-        <cylinder radius="0.05" length="0.5"/>
-      </geometry>
-      <origin xyz="0 0 0"/>
-    </collision>
-    <xacro:cylinder_inertia m="5" r="0.05" h="0.5" />
+        <cylinder radius="0.05" length="0.75"/>
+      </geometry>
+      <origin xyz="0 0 0"/>
+    </visual>
+    <collision>
+      <geometry>
+        <cylinder radius="0.05" length="0.75"/>
+      </geometry>
+      <origin xyz="0 0 0"/>
+    </collision>
+    <xacro:cylinder_inertia m="5" r="0.05" h="0.75" />
   </link>
   <joint name="pole_holder_to_pole" type="fixed">

Commit message: Add new effort limits

File: src/cart_pole/cart_pole_bringup/urdf/cart_pole.urdf.xacro (robot description, xacro)
@@ -85,5 +85,5 @@
     <parent link="pole_holder"/>
     <child link="pole_holder2"/>
-    <limit effort="10" lower="-1.57" upper="1.57" velocity="15"/>
+    <limit effort="1000" lower="-1.57" upper="1.57" velocity="100"/>
   </joint>
   <link name="pole">
@@ -189,7 +189,7 @@
     </hardware>
     <joint name="slider_to_cart">
-      <command_interface name="velocity">
-        <param name="min">-15</param>
-        <param name="max">15</param>
+      <command_interface name="effort">
+        <param name="min">-1000</param>
+        <param name="max">1000</param>
       </command_interface>
       <state_interface name="velocity"/>

Commit message: Urdf refactor. Use better naming and consistent convention

File: src/cart_pole/cart_pole_bringup/urdf/cart_pole.urdf.xacro (robot description, xacro)
@@ -4,165 +4,165 @@
     <inertial>
       <origin xyz="0 0 0" rpy="${pi/2} 0 0" />
-      <mass value="${m}"/>
-      <inertia ixx="${(m/12) * (3*r*r + h*h)}" ixy = "0" ixz = "0" iyy="${(m/12) * (3*r*r + h*h)}" iyz = "0" izz="${(m/2) * (r*r)}"/>
+      <mass value="${m}" />
+      <inertia ixx="${(m/12) * (3*r*r + h*h)}" ixy = "0" ixz = "0" iyy="${(m/12) * (3*r*r + h*h)}" iyz = "0" izz="${(m/2) * (r*r)}" />
     </inertial>
   </xacro:macro>
-  <link name="world"/>
+  <link name="world" />
   <link name="slideBar">
     <visual>
-      <geometry>
-        <box size="10 0.05 0.05"/>
-      </geometry>
-      <origin xyz="0 0 1"/>
-    </visual>
-    <inertial>
-      <mass value="100"/>
-      <inertia ixx="1" ixy="0" ixz="0" iyy="1" iyz="0" izz="1"/>
+      <origin xyz="0 0 1" />
+      <geometry>
+        <box size="10 0.05 0.05" />
+      </geometry>
+    </visual>
+    <inertial>
+      <mass value="100" />
+      <inertia ixx="1" ixy="0" ixz="0" iyy="1" iyz="0" izz="1" />
     </inertial>
   </link>
   <link name="cart">
     <visual>
-      <geometry>
-        <box size="0.5 0.5 0.2"/>
-      </geometry>
-      <origin xyz="0 0 0"/>
-    </visual>
-    <collision>
-      <geometry>
-        <box size="0.5 0.5 0.2"/>
-      </geometry>
-      <origin xyz="0 0 0"/>
-    </collision>
-    <inertial>
-      <mass value="1"/>
-      <inertia ixx="1" ixy="0" ixz="0" iyy="1" iyz="0" izz="1"/>
-    </inertial>
-  </link>
+      <origin xyz="0 0 0" />
+      <geometry>
+        <box size="0.5 0.5 0.2" />
+      </geometry>
+    </visual>
+    <collision>
+      <origin xyz="0 0 0" />
+      <geometry>
+        <box size="0.5 0.5 0.2" />
+      </geometry>
+    </collision>
+    <inertial>
+      <mass value="1" />
+      <inertia ixx="1" ixy="0" ixz="0" iyy="1" iyz="0" izz="1" />
+    </inertial>
+  </link>
+  <link name="pole_holder_base">
+    <visual>
+      <origin xyz="0 0 0" />
+      <geometry>
+        <box size="0.1 0.1 0.2" />
+      </geometry>
+    </visual>
+    <collision>
+      <origin xyz="0 0 0" />
+      <geometry>
+        <box size="0.1 0.1 0.2" />
+      </geometry>
+    </collision>
+    <inertial>
+      <mass value="1" />
+      <inertia ixx="1" ixy="0" ixz="0" iyy="1" iyz="0" izz="1" />
+    </inertial>
+  </link>
+  <joint name="cart_to_pole_holder_base" type="fixed">
+    <origin xyz="0 0 0.2" />
+    <parent link="cart" />
+    <child link="pole_holder" />
+  </joint>
   <link name="pole_holder">
     <visual>
-      <origin xyz="0 0 0"/>
-      <geometry>
-        <box size="0.1 0.1 0.2"/>
-      </geometry>
-    </visual>
-    <collision>
-      <geometry>
-        <box size="0.1 0.1 0.2"/>
-      </geometry>
-      <origin xyz="0 0 0"/>
-    </collision>
-    <inertial>
-      <mass value="1"/>
-      <inertia ixx="1" ixy="0" ixz="0" iyy="1" iyz="0" izz="1"/>
-    </inertial>
-  </link>
-  <joint name="cart_to_pole_holder" type="fixed">
-    <origin xyz="0 0 0.2"/>
-    <parent link="cart"/>
-    <child link="pole_holder"/>
-  </joint>
-  <link name="pole_holder2">
-    <visual>
-      <geometry>
-        <cylinder radius="0.05" length="0.05"/>
-      </geometry>
-      <origin xyz="0 0 0" rpy="1.57 0 0"/>
-    </visual>
-    <collision>
-      <geometry>
-        <cylinder radius="0.05" length="0.05"/>
-      </geometry>
-      <origin xyz="0 0 0" rpy="1.57 0 0"/>
-    </collision>
-    <inertial>
-      <mass value="1.5"/>
-      <inertia ixx="1" ixy="0" ixz="0" iyy="1" iyz="0" izz="1"/>
+      <origin xyz="0 0 0" rpy="1.57 0 0" />
+      <geometry>
+        <cylinder radius="0.05" length="0.05" />
+      </geometry>
+    </visual>
+    <collision>
+      <origin xyz="0 0 0" rpy="1.57 0 0" />
+      <geometry>
+        <cylinder radius="0.05" length="0.05" />
+      </geometry>
+    </collision>
+    <inertial>
+      <mass value="1.5" />
+      <inertia ixx="1" ixy="0" ixz="0" iyy="1" iyz="0" izz="1" />
     </inertial>
   </link>
   <joint name="pole_holder_to_pole_holder2" type="revolute">
-    <axis xyz="0 1 0"/>
+    <axis xyz="0 1 0" />
     <origin xyz="0 0.075 0.05" rpy="0 0.001 0" />
-    <parent link="pole_holder"/>
-    <child link="pole_holder2"/>
-    <limit effort="1000" lower="-1.57" upper="1.57" velocity="100"/>
+    <parent link="pole_holder_base" />
+    <child link="pole_holder" />
+    <limit effort="1000" lower="-1.57" upper="1.57" velocity="100" />
   </joint>
   <link name="pole">
     <visual>
-      <geometry>
-        <cylinder radius="0.05" length="0.75"/>
-      </geometry>
-      <origin xyz="0 0 0"/>
-    </visual>
-    <collision>
-      <geometry>
-        <cylinder radius="0.05" length="0.75"/>
-      </geometry>
-      <origin xyz="0 0 0"/>
+      <origin xyz="0 0 0" />
+      <geometry>
+        <cylinder radius="0.05" length="0.75" />
+      </geometry>
+    </visual>
+    <collision>
+      <origin xyz="0 0 0" />
+      <geometry>
+        <cylinder radius="0.05" length="0.75" />
+      </geometry>
     </collision>
     <xacro:cylinder_inertia m="5" r="0.05" h="0.75" />
   </link>
   <joint name="pole_holder_to_pole" type="fixed">
-    <origin xyz="0 0.075 0.15"/>
-    <parent link="pole_holder2"/>
-    <child link="pole"/>
+    <origin xyz="0 0.075 0.15" />
+    <parent link="pole_holder2" />
+    <child link="pole" />
   </joint>
   <link name="leg1">
     <visual>
-      <geometry>
-        <cylinder radius="0.2" length="2.0"/>
-      </geometry>
-      <origin xyz="0 0 0"/>
-    </visual>
-    <collision>
-      <geometry>
-        <cylinder radius="0.2" length="2.0"/>
-      </geometry>
-      <origin xyz="0 0 0"/>
-    </collision>
-    <inertial>
-      <mass value="2"/>
-      <inertia ixx="1" ixy="0" ixz="0" iyy="1" iyz="0" izz="1"/>
+      <origin xyz="0 0 0" />
+      <geometry>
+        <cylinder radius="0.2" length="2.0" />
+      </geometry>
+    </visual>
+    <collision>
+      <origin xyz="0 0 0" />
+      <geometry>
+        <cylinder radius="0.2" length="2.0" />
+      </geometry>
+    </collision>
+    <inertial>
+      <mass value="2" />
+      <inertia ixx="1" ixy="0" ixz="0" iyy="1" iyz="0" izz="1" />
     </inertial>
   </link>
   <link name="leg2">
     <visual>
-      <geometry>
-        <cylinder radius="0.2" length="2.0"/>
-      </geometry>
-      <origin xyz="0 0 0"/>
-    </visual>
-    <collision>
-      <geometry>
-        <cylinder radius="0.2" length="2.0"/>
-      </geometry>
-      <origin xyz="0 0 0"/>
-    </collision>
-    <inertial>
-      <mass value="2"/>
-      <inertia ixx="1" ixy="0" ixz="0" iyy="1" iyz="0" izz="1"/>
+      <origin xyz="0 0 0" />
+      <geometry>
+        <cylinder radius="0.2" length="2.0" />
+      </geometry>
+    </visual>
+    <collision>
+      <origin xyz="0 0 0" />
+      <geometry>
+        <cylinder radius="0.2" length="2.0" />
+      </geometry>
+    </collision>
+    <inertial>
+      <mass value="2" />
+      <inertia ixx="1" ixy="0" ixz="0" iyy="1" iyz="0" izz="1" />
     </inertial>
   </link>
   <joint name="world_to_base" type="fixed">
-    <origin rpy="0 0 0" xyz="0 0 1"/>
-    <parent link="world"/>
-    <child link="slideBar"/>
+    <origin rpy="0 0 0" xyz="0 0 1" />
+    <parent link="world" />
+    <child link="slideBar" />
   </joint>
   <joint name="slider_to_cart" type="prismatic">
-    <axis xyz="1 0 0"/>
-    <origin xyz="0 0 1.0"/>
-    <parent link="slideBar"/>
-    <child link="cart"/>
-    <limit effort="10.0" lower="-5" upper="5" velocity="30"/>
-    <dynamics damping="0.1" friction="0.1"/>
+    <axis xyz="1 0 0" />
+    <origin xyz="0 0 1.0" />
+    <parent link="slideBar" />
+    <child link="cart" />
+    <limit effort="10.0" lower="-5" upper="5" velocity="30" />
+    <dynamics damping="0.1" friction="0.1" />
   </joint>
   <joint name="slider_to_leg1" type="fixed">
-    <origin xyz="-5 0 1"/>
-    <parent link="slideBar"/>
-    <child link="leg1"/>
+    <origin xyz="-5 0 1" />
+    <parent link="slideBar" />
+    <child link="leg1" />
   </joint>
   <joint name="slider_to_leg2" type="fixed">
-    <origin xyz="5 0 1"/>
-    <parent link="slideBar"/>
-    <child link="leg2"/>
+    <origin xyz="5 0 1" />
+    <parent link="slideBar" />
+    <child link="leg2" />
   </joint>
   <gazebo reference="slideBar">
@@ -193,10 +193,10 @@
         <param name="max">1000</param>
       </command_interface>
-      <state_interface name="velocity"/>
-      <state_interface name="effort"/>
-      <state_interface name="position"/>
+      <state_interface name="velocity" />
+      <state_interface name="effort" />
+      <state_interface name="position" />
     </joint>
     <joint name="pole_holder_to_pole">
-      <state_interface name="velocity"/>
+      <state_interface name="velocity" />
       <state_interface name="position">
           <param name="initial_value">0.001</param>

Commit message: Add urdf macros file and fix urdf

File: src/cart_pole/cart_pole_bringup/urdf/cart_pole.urdf.xacro (robot description, xacro)
@@ -1,11 +1,5 @@
 <?xml version="1.0" ?>
 <robot name="cartopole" xmlns:xacro="http://ros.org/wiki/xacro">
-  <xacro:macro name="cylinder_inertia" params="m r h">
-    <inertial>
-      <origin xyz="0 0 0" rpy="${pi/2} 0 0" />
-      <mass value="${m}" />
-      <inertia ixx="${(m/12) * (3*r*r + h*h)}" ixy = "0" ixz = "0" iyy="${(m/12) * (3*r*r + h*h)}" iyz = "0" izz="${(m/2) * (r*r)}" />
-    </inertial>
-  </xacro:macro>
+  <xacro:include filename="$(find cart_pole_bringup)/urdf/macros.urdf.xacro" />
   <link name="world" />
   <link name="slideBar">
@@ -60,5 +54,5 @@
     <origin xyz="0 0 0.2" />
     <parent link="cart" />
-    <child link="pole_holder" />
+    <child link="pole_holder_base" />
   </joint>
   <link name="pole_holder">
@@ -80,5 +74,5 @@
     </inertial>
   </link>
-  <joint name="pole_holder_to_pole_holder2" type="revolute">
+  <joint name="pole_holder_base_to_pole_holder" type="revolute">
     <axis xyz="0 1 0" />
     <origin xyz="0 0.075 0.05" rpy="0 0.001 0" />
@@ -104,5 +98,5 @@
   <joint name="pole_holder_to_pole" type="fixed">
     <origin xyz="0 0.075 0.15" />
-    <parent link="pole_holder2" />
+    <parent link="pole_holder" />
     <child link="pole" />
   </joint>
