Commit message: Use cylinder inertia macro

File: src/cart_pole/cart_pole_bringup/urdf/cart_pole.urdf.xacro (robot description, xacro)
@@ -69,8 +69,5 @@
       </geometry>
     </collision>
-    <inertial>
-      <mass value="1.5" />
-      <inertia ixx="1" ixy="0" ixz="0" iyy="1" iyz="0" izz="1" />
-    </inertial>
+    <xacro:cylinder_inertia m="1.5" r="0.05" h="0.0.5" />
   </link>
   <joint name="pole_holder_base_to_pole_holder" type="revolute">
@@ -114,8 +111,5 @@
       </geometry>
     </collision>
-    <inertial>
-      <mass value="2" />
-      <inertia ixx="1" ixy="0" ixz="0" iyy="1" iyz="0" izz="1" />
-    </inertial>
+    <xacro:cylinder_inertia m="2" r="0.2" h="2.0" />
   </link>
   <link name="leg2">
@@ -132,8 +126,5 @@
       </geometry>
     </collision>
-    <inertial>
-      <mass value="2" />
-      <inertia ixx="1" ixy="0" ixz="0" iyy="1" iyz="0" izz="1" />
-    </inertial>
+    <xacro:cylinder_inertia m="2" r="0.2" h="2.0" />
   </link>
   <joint name="world_to_base" type="fixed">

Commit message: Rename leg1/2 to right/left limitter

File: src/cart_pole/cart_pole_bringup/urdf/cart_pole.urdf.xacro (robot description, xacro)
@@ -98,5 +98,5 @@
     <child link="pole" />
   </joint>
-  <link name="leg1">
+  <link name="left_limitter">
     <visual>
       <origin xyz="0 0 0" />
@@ -113,5 +113,5 @@
     <xacro:cylinder_inertia m="2" r="0.2" h="2.0" />
   </link>
-  <link name="leg2">
+  <link name="right_limitter">
     <visual>
       <origin xyz="0 0 0" />
@@ -135,19 +135,19 @@
   <joint name="slider_to_cart" type="prismatic">
     <axis xyz="1 0 0" />
-    <origin xyz="0 0 1.0" />
+    <origin xyz="0 0 1" />
     <parent link="slideBar" />
     <child link="cart" />
-    <limit effort="10.0" lower="-5" upper="5" velocity="30" />
+    <limit effort="10" lower="-5" upper="5" velocity="30" />
     <dynamics damping="0.1" friction="0.1" />
   </joint>
-  <joint name="slider_to_leg1" type="fixed">
+  <joint name="slider_to_left_limitter" type="fixed">
     <origin xyz="-5 0 1" />
     <parent link="slideBar" />
-    <child link="leg1" />
+    <child link="left_limitter" />
   </joint>
-  <joint name="slider_to_leg2" type="fixed">
+  <joint name="slider_to_right_limitter" type="fixed">
     <origin xyz="5 0 1" />
     <parent link="slideBar" />
-    <child link="leg2" />
+    <child link="right_limitter" />
   </joint>
   <gazebo reference="slideBar">

Commit message: Rename slideBar to slide_bar

File: src/cart_pole/cart_pole_bringup/urdf/cart_pole.urdf.xacro (robot description, xacro)
@@ -3,5 +3,5 @@
   <xacro:include filename="$(find cart_pole_bringup)/urdf/macros.urdf.xacro" />
   <link name="world" />
-  <link name="slideBar">
+  <link name="slide_bar">
     <visual>
       <origin xyz="0 0 1" />
@@ -10,8 +10,4 @@
       </geometry>
     </visual>
-    <inertial>
-      <mass value="100" />
-      <inertia ixx="1" ixy="0" ixz="0" iyy="1" iyz="0" izz="1" />
-    </inertial>
   </link>
   <link name="cart">
@@ -131,10 +127,10 @@
     <origin rpy="0 0 0" xyz="0 0 1" />
     <parent link="world" />
-    <child link="slideBar" />
+    <child link="slide_bar" />
   </joint>
   <joint name="slider_to_cart" type="prismatic">
     <axis xyz="1 0 0" />
     <origin xyz="0 0 1" />
-    <parent link="slideBar" />
+    <parent link="slide_bar" />
     <child link="cart" />
     <limit effort="10" lower="-5" upper="5" velocity="30" />
@@ -143,13 +139,13 @@
   <joint name="slider_to_left_limitter" type="fixed">
     <origin xyz="-5 0 1" />
-    <parent link="slideBar" />
+    <parent link="slide_bar" />
     <child link="left_limitter" />
   </joint>
   <joint name="slider_to_right_limitter" type="fixed">
     <origin xyz="5 0 1" />
-    <parent link="slideBar" />
+    <parent link="slide_bar" />
     <child link="right_limitter" />
   </joint>
-  <gazebo reference="slideBar">
+  <gazebo reference="slide_bar">
     <visual>
       <material>

Commit message: Use box inertia formula

File: src/cart_pole/cart_pole_bringup/urdf/cart_pole.urdf.xacro (robot description, xacro)
@@ -24,8 +24,5 @@
       </geometry>
     </collision>
-    <inertial>
-      <mass value="1" />
-      <inertia ixx="1" ixy="0" ixz="0" iyy="1" iyz="0" izz="1" />
-    </inertial>
+    <xacro:box_inertia m="1" w="0.5" h="0.2" d="0.5" />
   </link>
   <link name="pole_holder_base">
@@ -42,8 +39,5 @@
       </geometry>
     </collision>
-    <inertial>
-      <mass value="1" />
-      <inertia ixx="1" ixy="0" ixz="0" iyy="1" iyz="0" izz="1" />
-    </inertial>
+   <xacro:box_inertia m="0.5" w="0.1" h="0.2" d="0.1" />
   </link>
   <joint name="cart_to_pole_holder_base" type="fixed">

Commit message: Update moving joints in the ros2 hardware if

File: src/cart_pole/cart_pole_bringup/urdf/cart_pole.urdf.xacro (robot description, xacro)
@@ -172,5 +172,5 @@
       <state_interface name="position" />
     </joint>
-    <joint name="pole_holder_to_pole">
+    <joint name="pole_holder_base_to_pole_holder">
       <state_interface name="velocity" />
       <state_interface name="position">

Commit message: Remove color of slider

File: src/cart_pole/cart_pole_bringup/urdf/cart_pole.urdf.xacro (robot description, xacro)
@@ -141,13 +141,4 @@
     <child link="right_limitter" />
   </joint>
-  <gazebo reference="slide_bar">
-    <visual>
-      <material>
-        <ambient>0 0.8 0 1</ambient>
-        <diffuse>0 0.8 0 1</diffuse>
-        <specular>0 0.8 0 1</specular>
-      </material>
-    </visual>
-  </gazebo>
   <gazebo reference="cart">
     <visual>

Commit message: Remove slider limitter

File: src/cart_pole/cart_pole_bringup/urdf/cart_pole.urdf.xacro (robot description, xacro)
@@ -10,4 +10,11 @@
       </geometry>
     </visual>
+    <collision>
+      <origin xyz="0 0 0" />
+      <geometry>
+        <box size="10 0.05 0.05" />
+      </geometry>
+    </collision>
+    <xacro:box_inertia m="5" w="10" h="0.05" d="0.05" />
   </link>
   <link name="cart">
@@ -88,34 +95,4 @@
     <child link="pole" />
   </joint>
-  <link name="left_limitter">
-    <visual>
-      <origin xyz="0 0 0" />
-      <geometry>
-        <cylinder radius="0.2" length="2.0" />
-      </geometry>
-    </visual>
-    <collision>
-      <origin xyz="0 0 0" />
-      <geometry>
-        <cylinder radius="0.2" length="2.0" />
-      </geometry>
-    </collision>
-    <xacro:cylinder_inertia m="2" r="0.2" h="2.0" />
-  </link>
-  <link name="right_limitter">
-    <visual>
-      <origin xyz="0 0 0" />
-      <geometry>
-        <cylinder radius="0.2" length="2.0" />
-      </geometry>
-    </visual>
-    <collision>
-      <origin xyz="0 0 0" />
-      <geometry>
-        <cylinder radius="0.2" length="2.0" />
-      </geometry>
-    </collision>
-    <xacro:cylinder_inertia m="2" r="0.2" h="2.0" />
-  </link>
   <joint name="world_to_base" type="fixed">
     <origin rpy="0 0 0" xyz="0 0 1" />
@@ -125,19 +102,9 @@
   <joint name="slider_to_cart" type="prismatic">
     <axis xyz="1 0 0" />
-    <origin xyz="0 0 1" />
+    <origin xyz="0 0 1.15" />
     <parent link="slide_bar" />
     <child link="cart" />
     <limit effort="10" lower="-5" upper="5" velocity="30" />
     <dynamics damping="0.1" friction="0.1" />
-  </joint>
-  <joint name="slider_to_left_limitter" type="fixed">
-    <origin xyz="-5 0 1" />
-    <parent link="slide_bar" />
-    <child link="left_limitter" />
-  </joint>
-  <joint name="slider_to_right_limitter" type="fixed">
-    <origin xyz="5 0 1" />
-    <parent link="slide_bar" />
-    <child link="right_limitter" />
   </joint>
   <gazebo reference="cart">

Commit message: Attach pole directly to the cart

File: src/cart_pole/cart_pole_bringup/urdf/cart_pole.urdf.xacro (robot description, xacro)
@@ -33,24 +33,4 @@
     <xacro:box_inertia m="1" w="0.5" h="0.2" d="0.5" />
   </link>
-  <link name="pole_holder_base">
-    <visual>
-      <origin xyz="0 0 0" />
-      <geometry>
-        <box size="0.1 0.1 0.2" />
-      </geometry>
-    </visual>
-    <collision>
-      <origin xyz="0 0 0" />
-      <geometry>
-        <box size="0.1 0.1 0.2" />
-      </geometry>
-    </collision>
-   <xacro:box_inertia m="0.5" w="0.1" h="0.2" d="0.1" />
-  </link>
-  <joint name="cart_to_pole_holder_base" type="fixed">
-    <origin xyz="0 0 0.2" />
-    <parent link="cart" />
-    <child link="pole_holder_base" />
-  </joint>
   <link name="pole_holder">
     <visual>
@@ -70,6 +50,6 @@
   <joint name="pole_holder_base_to_pole_holder" type="revolute">
     <axis xyz="0 1 0" />
-    <origin xyz="0 0.075 0.05" rpy="0 0.001 0" />
-    <parent link="pole_holder_base" />
+    <origin xyz="0 0.28 0.05" rpy="0 0.001 0" />
+    <parent link="cart" />
     <child link="pole_holder" />
     <limit effort="1000" lower="-1.57" upper="1.57" velocity="100" />
@@ -91,5 +71,5 @@
   </link>
   <joint name="pole_holder_to_pole" type="fixed">
-    <origin xyz="0 0.075 0.15" />
+    <origin xyz="0 0.075 0.35" />
     <parent link="pole_holder" />
     <child link="pole" />

Commit message: Adjust simulation values

File: src/cart_pole/cart_pole_bringup/urdf/cart_pole.urdf.xacro (robot description, xacro)
@@ -16,5 +16,5 @@
       </geometry>
     </collision>
-    <xacro:box_inertia m="5" w="10" h="0.05" d="0.05" />
+    <xacro:box_inertia m="1" w="10" h="0.05" d="0.05" />
   </link>
   <link name="cart">
@@ -31,5 +31,5 @@
       </geometry>
     </collision>
-    <xacro:box_inertia m="1" w="0.5" h="0.2" d="0.5" />
+    <xacro:box_inertia m="0.4" w="0.5" h="0.2" d="0.5" />
   </link>
   <link name="pole_holder">
@@ -46,5 +46,5 @@
       </geometry>
     </collision>
-    <xacro:cylinder_inertia m="1" r="0.05" h="0.05" />
+    <xacro:cylinder_inertia m="0.001" r="0.05" h="0.05" />
   </link>
   <joint name="pole_holder_base_to_pole_holder" type="revolute">
@@ -53,5 +53,5 @@
     <parent link="cart" />
     <child link="pole_holder" />
-    <limit effort="1000" lower="-1.57" upper="1.57" velocity="100" />
+    <limit effort="10000" lower="-1.4" upper="1.4" velocity="1000" />
   </joint>
   <link name="pole">
@@ -68,5 +68,5 @@
       </geometry>
     </collision>
-    <xacro:cylinder_inertia m="2" r="0.05" h="0.75" />
+    <xacro:cylinder_inertia m="0.002" r="0.05" h="0.75" />
   </link>
   <joint name="pole_holder_to_pole" type="fixed">
@@ -85,6 +85,6 @@
     <parent link="slide_bar" />
     <child link="cart" />
-    <limit effort="10" lower="-5" upper="5" velocity="30" />
-    <dynamics damping="0.1" friction="0.1" />
+    <limit effort="10000" lower="-5" upper="5" velocity="1000" />
+    <dynamics damping="0.05" />
   </joint>
   <gazebo reference="cart">
@@ -102,8 +102,5 @@
     </hardware>
     <joint name="slider_to_cart">
-      <command_interface name="effort">
-        <param name="min">-1000</param>
-        <param name="max">1000</param>
-      </command_interface>
+      <command_interface name="effort" />
       <state_interface name="velocity" />
       <state_interface name="effort" />

Commit message: Remove ues of ros controll

File: src/cart_pole/cart_pole_bringup/urdf/cart_pole.urdf.xacro (robot description, xacro)
@@ -97,22 +97,3 @@
     </visual>
   </gazebo>
-  <ros2_control name="GazeboSimSystem" type="system">
-    <hardware>
-      <plugin>gz_ros2_control/GazeboSimSystem</plugin>
-    </hardware>
-    <joint name="slider_to_cart">
-      <command_interface name="effort" />
-      <state_interface name="effort" />
-    </joint>
-    <joint name="pole_holder_base_to_pole_holder">
-      <state_interface name="position">
-          <param name="initial_value">0.001</param>
-        </state_interface>
-    </joint>
-  </ros2_control>
-  <gazebo>
-    <plugin filename="gz_ros2_control-system" name="gz_ros2_control::GazeboSimROS2ControlPlugin">
-      <parameters>$(find cart_pole_bringup)/config/cart_pole_controllers.yaml</parameters>
-    </plugin>
-  </gazebo>
 </robot>

Commit message: Update inital pole pose

File: src/cart_pole/cart_pole_bringup/urdf/cart_pole.urdf.xacro (robot description, xacro)
@@ -50,5 +50,5 @@
   <joint name="pole_holder_base_to_pole_holder" type="revolute">
     <axis xyz="0 1 0" />
-    <origin xyz="0 0.28 0.05" rpy="0 0.001 0" />
+    <origin xyz="0 0.28 0.05" rpy="0 0 0" />
     <parent link="cart" />
     <child link="pole_holder" />

Commit message: Fixed inertia and collision
Signed-off-by: Jakub Delicat <delicat.kuba@gmail.com>

File: src/cart_pole/cart_pole_bringup/urdf/cart_pole.urdf.xacro (robot description, xacro)
@@ -11,10 +11,10 @@
     </visual>
     <collision>
-      <origin xyz="0 0 0" />
+      <origin xyz="0 0 1" />
       <geometry>
         <box size="10 0.05 0.05" />
       </geometry>
     </collision>
-    <xacro:box_inertia m="1" w="10" h="0.05" d="0.05" />
+    <xacro:box_inertia m="1" w="10" h="0.05" d="0.05"  xyz="0 0 1" />
   </link>
   <link name="cart">
@@ -31,5 +31,5 @@
       </geometry>
     </collision>
-    <xacro:box_inertia m="0.4" w="0.5" h="0.2" d="0.5" />
+    <xacro:box_inertia m="0.4" w="0.5" h="0.5" d="0.2" />
   </link>
   <link name="pole_holder">
@@ -46,5 +46,5 @@
       </geometry>
     </collision>
-    <xacro:cylinder_inertia m="0.001" r="0.05" h="0.05" />
+    <xacro:cylinder_inertia m="0.001" r="0.05" h="0.05" rpy="1.57 0 0" />
   </link>
   <joint name="pole_holder_base_to_pole_holder" type="revolute">

File: src/cart_pole/cart_pole_bringup/urdf/macros.urdf.xacro (robot description, xacro)
@@ -1,14 +1,14 @@
 <?xml version="1.0"?>
 <robot name="cart_pole" xmlns:xacro="http://ros.org/wiki/xacro">
-  <xacro:macro name="box_inertia" params="m w h d">
+  <xacro:macro name="box_inertia" params="m w h d xyz:='0.0 0.0 0.0' rpy:='0.0 0.0 0.0'">
     <inertial>
-      <origin xyz="0 0 0" rpy="${pi/2} 0 ${pi/2}"/>
+      <origin xyz="${xyz}" rpy="${rpy}"/>
       <mass value="${m}"/>
       <inertia ixx="${(m/12) * (h*h + d*d)}" ixy="0.0" ixz="0.0" iyy="${(m/12) * (w*w + d*d)}" iyz="0.0" izz="${(m/12) * (w*w + h*h)}"/>
     </inertial>
   </xacro:macro>
-  <xacro:macro name="cylinder_inertia" params="m r h">
+  <xacro:macro name="cylinder_inertia" params="m r h xyz:='0.0 0.0 0.0' rpy:='0.0 0.0 0.0'">
     <inertial>
-      <origin xyz="0 0 0" rpy="${pi/2} 0 0" />
+      <origin xyz="${xyz}" rpy="${rpy}"/>
       <mass value="${m}"/>
       <inertia ixx="${(m/12) * (3*r*r + h*h)}" ixy = "0" ixz = "0" iyy="${(m/12) * (3*r*r + h*h)}" iyz = "0" izz="${(m/2) * (r*r)}"/>

Commit message: Added 010 cart pole
Signed-off-by: Jakub Delicat <delicat.kuba@gmail.com>

File: src/cart_pole/cart_pole_bringup/urdf/cart_pole.urdf.xacro (robot description, xacro)
@@ -5,16 +5,16 @@
   <link name="slide_bar">
     <visual>
-      <origin xyz="0 0 1" />
+      <origin xyz="0 0 0" />
       <geometry>
-        <box size="10 0.05 0.05" />
+        <mesh filename="package://cart_pole_bringup/meshes/slide_bar.dae"  />
       </geometry>
     </visual>
     <collision>
-      <origin xyz="0 0 1" />
+      <origin xyz="0 0 0" />
       <geometry>
         <box size="10 0.05 0.05" />
       </geometry>
     </collision>
-    <xacro:box_inertia m="1" w="10" h="0.05" d="0.05"  xyz="0 0 1" />
+    <xacro:box_inertia m="10" w="2" h="0.05" d="0.05"  xyz="0 0 0" rpy="0 0 ${pi/2.0}" />
   </link>
   <link name="cart">
@@ -22,5 +22,5 @@
       <origin xyz="0 0 0" />
       <geometry>
-        <box size="0.5 0.5 0.2" />
+        <mesh filename="package://cart_pole_bringup/meshes/cart.dae" />
       </geometry>
     </visual>
@@ -31,59 +31,54 @@
       </geometry>
     </collision>
-    <xacro:box_inertia m="0.4" w="0.5" h="0.5" d="0.2" />
+    <inertial>
+      <origin xyz="0 0 0" rpy="0 0 0"/>
+      <mass value="1.006"/>
+      <!-- TODO: @delipl wrong inertia here -->
+      <inertia
+          ixx="0.000199325" ixy="2.051e-06"     ixz="-7.69e-06"
+                            iyy="0.002043291"  iyz="-1.714e-06"
+                                              izz="0.002188884"
+      />
+    </inertial>
   </link>
-  <link name="pole_holder">
+  <link name="pole_with_holder">
     <visual>
-      <origin xyz="0 0 0" rpy="1.57 0 0" />
+      <origin xyz="0 0 0" rpy="0 0 0" />
       <geometry>
-        <cylinder radius="0.05" length="0.05" />
+        <mesh filename="package://cart_pole_bringup/meshes/pole_with_holder.dae"  />
       </geometry>
     </visual>
     <collision>
-      <origin xyz="0 0 0" rpy="1.57 0 0" />
+      <origin xyz="0 0 0" rpy="0 0 0" />
       <geometry>
         <cylinder radius="0.05" length="0.05" />
       </geometry>
     </collision>
-    <xacro:cylinder_inertia m="0.001" r="0.05" h="0.05" rpy="1.57 0 0" />
+    <inertial>
+      <origin xyz="0.04 0.435057 0" rpy="0 0 0"/>
+      <mass value="0.455"/>
+      <inertia ixx="0.044100482" ixy="-0.000237859" ixz="-0.000004"
+                                 iyy="0.000040196"  iyz="-0.000037"
+                                                    izz="0.044096759" />
+    </inertial>
   </link>
-  <joint name="pole_holder_base_to_pole_holder" type="revolute">
-    <axis xyz="0 1 0" />
-    <origin xyz="0 0.28 0.05" rpy="0 0 0" />
+  <joint name="slide_to_pole_with_holder" type="revolute">
+    <axis xyz="1 0 0" />
+    <origin xyz="0.10161 0 0" rpy="${pi/2} 0 0" />
     <parent link="cart" />
-    <child link="pole_holder" />
+    <child link="pole_with_holder" />
     <limit effort="10000" lower="-1.4" upper="1.4" velocity="1000" />
   </joint>
-  <link name="pole">
-    <visual>
-      <origin xyz="0 0 0" />
-      <geometry>
-        <cylinder radius="0.05" length="0.75" />
-      </geometry>
-    </visual>
-    <collision>
-      <origin xyz="0 0 0" />
-      <geometry>
-        <cylinder radius="0.05" length="0.75" />
-      </geometry>
-    </collision>
-    <xacro:cylinder_inertia m="0.002" r="0.05" h="0.75" />
-  </link>
-  <joint name="pole_holder_to_pole" type="fixed">
-    <origin xyz="0 0.075 0.35" />
-    <parent link="pole_holder" />
-    <child link="pole" />
-  </joint>
   <joint name="world_to_base" type="fixed">
-    <origin rpy="0 0 0" xyz="0 0 1" />
+    <origin rpy="0 0 ${pi}" xyz="0 0 1" />
     <parent link="world" />
     <child link="slide_bar" />
   </joint>
   <joint name="slider_to_cart" type="prismatic">
-    <axis xyz="1 0 0" />
-    <origin xyz="0 0 1.15" />
+    <axis xyz="0 -1 0" />
+    <origin xyz="0.09 ${0.435057 - 0.435057} 0.004" />
     <parent link="slide_bar" />
     <child link="cart" />
-    <limit effort="10000" lower="-5" upper="5" velocity="1000" />
+    <limit effort="10000" lower="${-0.133 - 0.435057}" upper="${1.21 - 0.435057}" velocity="1000" />
     <dynamics damping="0.05" />
   </joint>
@@ -94,4 +89,13 @@
         <diffuse>0 0 0.8 1</diffuse>
         <specular>0 0 0.8 1</specular>
+      </material>
+    </visual>
+  </gazebo>
+  <gazebo reference="pole_with_holder">
+    <visual>
+      <material>
+        <ambient>0.8 0 0 1</ambient>
+        <diffuse>0.8 0 0 1</diffuse>
+        <specular>0.8 0 0 1</specular>
       </material>
     </visual>
@@ -106,5 +110,5 @@
       <topic>joint_states</topic>
       <joint_name>slider_to_cart</joint_name>
-      <joint_name>pole_holder_base_to_pole_holder</joint_name>
+      <joint_name>slide_to_pole_with_holder</joint_name>
     </plugin>
   </gazebo>

Commit message: Fixed inertia and collisions | added cart state to output
Signed-off-by: Jakub Delicat <delicat.kuba@gmail.com>

File: src/cart_pole/cart_pole_bringup/urdf/cart_pole.urdf.xacro (robot description, xacro)
@@ -11,10 +11,10 @@
     </visual>
     <collision>
-      <origin xyz="0 0 0" />
+      <origin xyz="0.025 -0.1 0" rpy="0 0 ${pi/2.0}" />
       <geometry>
-        <box size="10 0.05 0.05" />
+        <box size="1.8 0.1 0.05" />
       </geometry>
     </collision>
-    <xacro:box_inertia m="10" w="2" h="0.05" d="0.05"  xyz="0 0 0" rpy="0 0 ${pi/2.0}" />
+    <xacro:box_inertia m="10" w="1.8" h="0.1" d="0.05"  xyz="0.025 -0.1 0" rpy="0 0 ${pi/2.0}" />
   </link>
   <link name="cart">
@@ -26,18 +26,14 @@
     </visual>
     <collision>
-      <origin xyz="0 0 0" />
+      <origin xyz="0.015 0 0" />
       <geometry>
-        <box size="0.5 0.5 0.2" />
+        <box size="0.16 0.16 0.11" />
       </geometry>
     </collision>
     <inertial>
-      <origin xyz="0 0 0" rpy="0 0 0"/>
-      <mass value="1.006"/>
-      <!-- TODO: @delipl wrong inertia here -->
-      <inertia
-          ixx="0.000199325" ixy="2.051e-06"     ixz="-7.69e-06"
-                            iyy="0.002043291"  iyz="-1.714e-06"
-                                              izz="0.002188884"
-      />
+      <mass value="1.006" />
+      <inertia ixx="0.001999325" ixy="0.00000769" ixz="0.000002051"
+                                 iyy="0.00218888" iyz="0.000001714"
+                                                  izz="0.002943291" />
     </inertial>
   </link>
@@ -50,11 +46,11 @@
     </visual>
     <collision>
-      <origin xyz="0 0 0" rpy="0 0 0" />
+      <origin xyz="0.04 0.485 0" rpy="${pi/2.0} 0 0" />
       <geometry>
-        <cylinder radius="0.05" length="0.05" />
+        <cylinder radius="0.01" length="1.0" />
       </geometry>
     </collision>
     <inertial>
-      <origin xyz="0.04 0.435057 0" rpy="0 0 0"/>
+      <origin xyz="0.039298 0.435057 0" rpy="0 0 0"/>
       <mass value="0.455"/>
       <inertia ixx="0.044100482" ixy="-0.000237859" ixz="-0.000004"
@@ -65,5 +61,5 @@
   <joint name="slide_to_pole_with_holder" type="revolute">
     <axis xyz="1 0 0" />
-    <origin xyz="0.10161 0 0" rpy="${pi/2} 0 0" />
+    <origin xyz="0.08 0 0" rpy="${pi/2} 0 0" />
     <parent link="cart" />
     <child link="pole_with_holder" />
