Commit message: Revert "Merge pull request #10 from delipl/main"
This reverts commit e80f65bed87299739876c92b21c7de15909c14a5, reversing
changes made to 03a0a12a7e1342bf6b63cca90b1f9ae801f6514d.

File: src/cart_pole/cart_pole_bringup/urdf/cart_pole.urdf.xacro (robot description, xacro)
@@ -5,16 +5,16 @@
   <link name="slide_bar">
     <visual>
-      <origin xyz="0 0 0" />
+      <origin xyz="0 0 1" />
       <geometry>
-        <mesh filename="package://cart_pole_bringup/meshes/slide_bar.dae"  />
+        <box size="10 0.05 0.05" />
       </geometry>
     </visual>
     <collision>
-      <origin xyz="0.025 -0.1 0" rpy="0 0 ${pi/2.0}" />
+      <origin xyz="0 0 1" />
       <geometry>
-        <box size="1.8 0.1 0.05" />
+        <box size="10 0.05 0.05" />
       </geometry>
     </collision>
-    <xacro:box_inertia m="10" w="1.8" h="0.1" d="0.05"  xyz="0.025 -0.1 0" rpy="0 0 ${pi/2.0}" />
+    <xacro:box_inertia m="1" w="10" h="0.05" d="0.05"  xyz="0 0 1" />
   </link>
   <link name="cart">
@@ -22,59 +22,68 @@
       <origin xyz="0 0 0" />
       <geometry>
-        <mesh filename="package://cart_pole_bringup/meshes/cart.dae" />
+        <box size="0.5 0.5 0.2" />
       </geometry>
     </visual>
     <collision>
-      <origin xyz="0.015 0 0" />
+      <origin xyz="0 0 0" />
       <geometry>
-        <box size="0.16 0.16 0.11" />
+        <box size="0.5 0.5 0.2" />
       </geometry>
     </collision>
-    <inertial>
-      <mass value="1.006" />
-      <inertia ixx="0.001999325" ixy="0.00000769" ixz="0.000002051"
-                                 iyy="0.00218888" iyz="0.000001714"
-                                                  izz="0.002943291" />
-    </inertial>
+    <xacro:box_inertia m="0.4" w="0.5" h="0.5" d="0.2" />
   </link>
-  <link name="pole_with_holder">
+  <link name="pole_holder">
     <visual>
-      <origin xyz="0 0 0" rpy="0 0 0" />
+      <origin xyz="0 0 0" rpy="1.57 0 0" />
       <geometry>
-        <mesh filename="package://cart_pole_bringup/meshes/pole_with_holder.dae"  />
+        <cylinder radius="0.05" length="0.05" />
       </geometry>
     </visual>
     <collision>
-      <origin xyz="0.04 0.485 0" rpy="${pi/2.0} 0 0" />
+      <origin xyz="0 0 0" rpy="1.57 0 0" />
       <geometry>
-        <cylinder radius="0.01" length="1.0" />
+        <cylinder radius="0.05" length="0.05" />
       </geometry>
     </collision>
-    <inertial>
-      <origin xyz="0.039298 0.435057 0" rpy="0 0 0"/>
-      <mass value="0.455"/>
-      <inertia ixx="0.044100482" ixy="-0.000237859" ixz="-0.000004"
-                                 iyy="0.000040196"  iyz="-0.000037"
-                                                    izz="0.044096759" />
-    </inertial>
+    <xacro:cylinder_inertia m="0.001" r="0.05" h="0.05" rpy="1.57 0 0" />
   </link>
-  <joint name="slide_to_pole_with_holder" type="revolute">
-    <axis xyz="1 0 0" />
-    <origin xyz="0.08 0 0" rpy="${pi/2} 0 0" />
+  <joint name="pole_holder_base_to_pole_holder" type="revolute">
+    <axis xyz="0 1 0" />
+    <origin xyz="0 0.28 0.05" rpy="0 0 0" />
     <parent link="cart" />
-    <child link="pole_with_holder" />
+    <child link="pole_holder" />
     <limit effort="10000" lower="-1.4" upper="1.4" velocity="1000" />
   </joint>
+  <link name="pole">
+    <visual>
+      <origin xyz="0 0 0" />
+      <geometry>
+        <cylinder radius="0.05" length="0.75" />
+      </geometry>
+    </visual>
+    <collision>
+      <origin xyz="0 0 0" />
+      <geometry>
+        <cylinder radius="0.05" length="0.75" />
+      </geometry>
+    </collision>
+    <xacro:cylinder_inertia m="0.002" r="0.05" h="0.75" />
+  </link>
+  <joint name="pole_holder_to_pole" type="fixed">
+    <origin xyz="0 0.075 0.35" />
+    <parent link="pole_holder" />
+    <child link="pole" />
+  </joint>
   <joint name="world_to_base" type="fixed">
-    <origin rpy="0 0 ${pi}" xyz="0 0 1" />
+    <origin rpy="0 0 0" xyz="0 0 1" />
     <parent link="world" />
     <child link="slide_bar" />
   </joint>
   <joint name="slider_to_cart" type="prismatic">
-    <axis xyz="0 -1 0" />
-    <origin xyz="0.09 ${0.435057 - 0.435057} 0.004" />
+    <axis xyz="1 0 0" />
+    <origin xyz="0 0 1.15" />
     <parent link="slide_bar" />
     <child link="cart" />
-    <limit effort="10000" lower="${-0.133 - 0.435057}" upper="${1.21 - 0.435057}" velocity="1000" />
+    <limit effort="10000" lower="-5" upper="5" velocity="1000" />
     <dynamics damping="0.05" />
   </joint>
@@ -85,13 +94,4 @@
         <diffuse>0 0 0.8 1</diffuse>
         <specular>0 0 0.8 1</specular>
-      </material>
-    </visual>
-  </gazebo>
-  <gazebo reference="pole_with_holder">
-    <visual>
-      <material>
-        <ambient>0.8 0 0 1</ambient>
-        <diffuse>0.8 0 0 1</diffuse>
-        <specular>0.8 0 0 1</specular>
       </material>
     </visual>
@@ -106,5 +106,5 @@
       <topic>joint_states</topic>
       <joint_name>slider_to_cart</joint_name>
-      <joint_name>slide_to_pole_with_holder</joint_name>
+      <joint_name>pole_holder_base_to_pole_holder</joint_name>
     </plugin>
   </gazebo>

Commit message: Adjust cart pole collision

File: src/cart_pole/cart_pole_bringup/urdf/cart_pole.urdf.xacro (robot description, xacro)
@@ -26,7 +26,7 @@
     </visual>
     <collision>
-      <origin xyz="0.015 0 0" />
+      <origin xyz="0.04 0 0" />
       <geometry>
-        <box size="0.16 0.16 0.11" />
+        <box size="0.1 0.16 0.11" />
       </geometry>
     </collision>

Commit message: Fix slider_to_pole joint's name

File: src/cart_pole/cart_pole_bringup/urdf/cart_pole.urdf.xacro (robot description, xacro)
@@ -59,5 +59,5 @@
     </inertial>
   </link>
-  <joint name="slide_to_pole_with_holder" type="revolute">
+  <joint name="slider_to_pole_with_holder" type="revolute">
     <axis xyz="1 0 0" />
     <origin xyz="0.08 0 0" rpy="${pi/2} 0 0" />
@@ -106,5 +106,5 @@
       <topic>joint_states</topic>
       <joint_name>slider_to_cart</joint_name>
-      <joint_name>slide_to_pole_with_holder</joint_name>
+      <joint_name>slider_to_pole_with_holder</joint_name>
     </plugin>
   </gazebo>

Commit message: Add pre-commit badge

File: src/cart_pole/cart_pole_bringup/urdf/cart_pole.urdf.xacro (robot description, xacro)
@@ -61,5 +61,5 @@
   <joint name="slider_to_pole_with_holder" type="revolute">
     <axis xyz="1 0 0" />
-    <origin xyz="0.08 0 0" rpy="${pi/2} 0 0" />
+    <origin xyz="0.05 0 0" rpy="${pi/2} 0 0" />
     <parent link="cart" />
     <child link="pole_with_holder" />
